File: hardware/led-strip-controller-esp8266/led-strip-controller-esp8266.kicad_pcb (KiCad board)
At the start: 2 copper layers, 16 parts, among them J1 Conn_01x04, J2 Conn_01x04, J3 Conn_01x04, Q1 IRLZ44N, Q2 IRLZ44N, Q3 IRLZ44N, Q4 IRLZ44N, Q5 IRLZ44N, Q6 IRLZ44N, Q7 IRLZ44N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

Commit message: More work on the schematic.
Connections:
- net /TRIGGER renamed Trigger
- U2 pad 28: +3V3 -> Net-(U2-Pad28)
Changed lines of the file:
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@@
     (zones 0)
     (modules 16)
-    (nets 48)
+    (nets 49)
   )
   (page A4)
@@
   (net 26 "Net-(U1-Pad18)")
   (net 27 "Net-(U1-PadPAD)")
-  (net 28 /TRIGGER)
-  (net 29 /LED0.0)
-  (net 30 "Net-(J1-Pad2)")
-  (net 31 "Net-(J1-Pad3)")
-  (net 32 /LED0.1)
-  (net 33 /LED0.2)
-  (net 34 "Net-(J1-Pad4)")
-  (net 35 "Net-(J3-Pad2)")
-  (net 36 /LED2.0)
-  (net 37 /LED2.1)
-  (net 38 "Net-(J3-Pad3)")
-  (net 39 "Net-(J3-Pad4)")
-  (net 40 /LED2.2)
-  (net 41 /LED1.0)
-  (net 42 "Net-(J2-Pad2)")
-  (net 43 "Net-(J2-Pad3)")
-  (net 44 /LED1.1)
-  (net 45 /LED1.2)
-  (net 46 "Net-(J2-Pad4)")
-  (net 47 +12V)
+  (net 28 /LED0.0)
+  (net 29 "Net-(J1-Pad2)")
+  (net 30 "Net-(J1-Pad3)")
+  (net 31 /LED0.1)
+  (net 32 /LED0.2)
+  (net 33 "Net-(J1-Pad4)")
+  (net 34 "Net-(J3-Pad2)")
+  (net 35 /LED2.0)
+  (net 36 /LED2.1)
+  (net 37 "Net-(J3-Pad3)")
+  (net 38 "Net-(J3-Pad4)")
+  (net 39 /LED2.2)
+  (net 40 /LED1.0)
+  (net 41 "Net-(J2-Pad2)")
+  (net 42 "Net-(J2-Pad3)")
+  (net 43 /LED1.1)
+  (net 44 /LED1.2)
+  (net 45 "Net-(J2-Pad4)")
+  (net 46 +12V)
+  (net 47 Trigger)
+  (net 48 "Net-(U2-Pad28)")
   (net_class Default "This is the default net class."
     (clearance 0.2)
@@
     (add_net /SCL)
     (add_net /SDA)
-    (add_net /TRIGGER)
     (add_net GND)
     (add_net "Net-(J1-Pad2)")
@@
     (add_net "Net-(U2-Pad20)")
     (add_net "Net-(U2-Pad21)")
+    (add_net "Net-(U2-Pad28)")
+    (add_net Trigger)
   )
   (module Connector_PinHeader_1.00mm:PinHeader_1x04_P1.00mm_Vertical (layer F.Cu)
@@
     )
     (pad 1 thru_hole rect (at 0 0 180) (size 0.85 0.85) (drill 0.5) (layers *.Cu *.Mask)
-      (net 47 +12V))
+      (net 46 +12V))
     (pad 2 thru_hole oval (at 0 1 180) (size 0.85 0.85) (drill 0.5) (layers *.Cu *.Mask)
-      (net 35 "Net-(J3-Pad2)"))
+      (net 34 "Net-(J3-Pad2)"))
     (pad 3 thru_hole oval (at 0 2 180) (size 0.85 0.85) (drill 0.5) (layers *.Cu *.Mask)
-      (net 38 "Net-(J3-Pad3)"))
+      (net 37 "Net-(J3-Pad3)"))
     (pad 4 thru_hole oval (at 0 3 180) (size 0.85 0.85) (drill 0.5) (layers *.Cu *.Mask)
-      (net 39 "Net-(J3-Pad4)"))
+      (net 38 "Net-(J3-Pad4)"))
     (model ${KISYS3DMOD}/Connector_PinHeader_1.00mm.3dshapes/PinHeader_1x04_P1.00mm_Vertical.wrl
       (at (xyz 0 0 0))
@@
     (fp_line (start -0.3175 -0.5) (end 0.635 -0.5) (layer F.Fab) (width 0.1))
     (pad 4 thru_hole oval (at 0 3 180) (size 0.85 0.85) (drill 0.5) (layers *.Cu *.Mask)
-      (net 46 "Net-(J2-Pad4)"))
+      (net 45 "Net-(J2-Pad4)"))
     (pad 3 thru_hole oval (at 0 2 180) (size 0.85 0.85) (drill 0.5) (layers *.Cu *.Mask)
-      (net 43 "Net-(J2-Pad3)"))
+      (net 42 "Net-(J2-Pad3)"))
     (pad 2 thru_hole oval (at 0 1 180) (size 0.85 0.85) (drill 0.5) (layers *.Cu *.Mask)
-      (net 42 "Net-(J2-Pad2)"))
+      (net 41 "Net-(J2-Pad2)"))
     (pad 1 thru_hole rect (at 0 0 180) (size 0.85 0.85) (drill 0.5) (layers *.Cu *.Mask)
-      (net 47 +12V))
+      (net 46 +12V))
     (model ${KISYS3DMOD}/Connector_PinHeader_1.00mm.3dshapes/PinHeader_1x04_P1.00mm_Vertical.wrl
       (at (xyz 0 0 0))
@@
     )
     (pad 1 thru_hole rect (at 0 0 180) (size 0.85 0.85) (drill 0.5) (layers *.Cu *.Mask)
-      (net 47 +12V))
+      (net 46 +12V))
     (pad 2 thru_hole oval (at 0 1 180) (size 0.85 0.85) (drill 0.5) (layers *.Cu *.Mask)
-      (net 30 "Net-(J1-Pad2)"))
+      (net 29 "Net-(J1-Pad2)"))
     (pad 3 thru_hole oval (at 0 2 180) (size 0.85 0.85) (drill 0.5) (layers *.Cu *.Mask)
-      (net 31 "Net-(J1-Pad3)"))
+      (net 30 "Net-(J1-Pad3)"))
     (pad 4 thru_hole oval (at 0 3 180) (size 0.85 0.85) (drill 0.5) (layers *.Cu *.Mask)
-      (net 34 "Net-(J1-Pad4)"))
+      (net 33 "Net-(J1-Pad4)"))
     (model ${KISYS3DMOD}/Connector_PinHeader_1.00mm.3dshapes/PinHeader_1x04_P1.00mm_Vertical.wrl
       (at (xyz 0 0 0))
@@
     )
     (pad 1 thru_hole rect (at 0 0 270) (size 1.905 2) (drill 1.1) (layers *.Cu *.Mask)
-      (net 40 /LED2.2))
+      (net 39 /LED2.2))
     (pad 2 thru_hole oval (at 2.54 0 270) (size 1.905 2) (drill 1.1) (layers *.Cu *.Mask)
-      (net 39 "Net-(J3-Pad4)"))
+      (net 38 "Net-(J3-Pad4)"))
     (pad 3 thru_hole oval (at 5.08 0 270) (size 1.905 2) (drill 1.1) (layers *.Cu *.Mask)
       (net 1 GND))
@@
       (net 1 GND))
     (pad 2 thru_hole oval (at 2.54 0 270) (size 1.905 2) (drill 1.1) (layers *.Cu *.Mask)
-      (net 38 "Net-(J3-Pad3)"))
+      (net 37 "Net-(J3-Pad3)"))
     (pad 1 thru_hole rect (at 0 0 270) (size 1.905 2) (drill 1.1) (layers *.Cu *.Mask)
-      (net 37 /LED2.1))
+      (net 36 /LED2.1))
     (model ${KISYS3DMOD}/Package_TO_SOT_THT.3dshapes/TO-220-3_Vertical.wrl
       (at (xyz 0 0 0))
@@
     )
     (pad 1 thru_hole rect (at 0 0 270) (size 1.905 2) (drill 1.1) (layers *.Cu *.Mask)
-      (net 36 /LED2.0))
+      (net 35 /LED2.0))
     (pad 2 thru_hole oval (at 2.54 0 270) (size 1.905 2) (drill 1.1) (layers *.Cu *.Mask)
-      (net 35 "Net-(J3-Pad2)"))
+      (net 34 "Net-(J3-Pad2)"))
     (pad 3 thru_hole oval (at 5.08 0 270) (size 1.905 2) (drill 1.1) (layers *.Cu *.Mask)
       (net 1 GND))
@@
       (net 1 GND))
     (pad 2 thru_hole oval (at 2.54 0 270) (size 1.905 2) (drill 1.1) (layers *.Cu *.Mask)
-      (net 46 "Net-(J2-Pad4)"))
+      (net 45 "Net-(J2-Pad4)"))
     (pad 1 thru_hole rect (at 0 0 270) (size 1.905 2) (drill 1.1) (layers *.Cu *.Mask)
-      (net 45 /LED1.2))
+      (net 44 /LED1.2))
     (model ${KISYS3DMOD}/Package_TO_SOT_THT.3dshapes/TO-220-3_Vertical.wrl
       (at (xyz 0 0 0))
@@
     )
     (pad 1 thru_hole rect (at 0 0 270) (size 1.905 2) (drill 1.1) (layers *.Cu *.Mask)
-      (net 44 /LED1.1))
+      (net 43 /LED1.1))
     (pad 2 thru_hole oval (at 2.54 0 270) (size 1.905 2) (drill 1.1) (layers *.Cu *.Mask)
-      (net 43 "Net-(J2-Pad3)"))
+      (net 42 "Net-(J2-Pad3)"))
     (pad 3 thru_hole oval (at 5.08 0 270) (size 1.905 2) (drill 1.1) (layers *.Cu *.Mask)
       (net 1 GND))
@@
       (net 1 GND))
     (pad 2 thru_hole oval (at 2.54 0 270) (size 1.905 2) (drill 1.1) (layers *.Cu *.Mask)
-      (net 42 "Net-(J2-Pad2)"))
+      (net 41 "Net-(J2-Pad2)"))
     (pad 1 thru_hole rect (at 0 0 270) (size 1.905 2) (drill 1.1) (layers *.Cu *.Mask)
-      (net 41 /LED1.0))
+      (net 40 /LED1.0))
     (model ${KISYS3DMOD}/Package_TO_SOT_THT.3dshapes/TO-220-3_Vertical.wrl
       (at (xyz 0 0 0))
@@
     )
     (pad 1 thru_hole rect (at 0 0 270) (size 1.905 2) (drill 1.1) (layers *.Cu *.Mask)
-      (net 33 /LED0.2))
+      (net 32 /LED0.2))
     (pad 2 thru_hole oval (at 2.54 0 270) (size 1.905 2) (drill 1.1) (layers *.Cu *.Mask)
-      (net 34 "Net-(J1-Pad4)"))
+      (net 33 "Net-(J1-Pad4)"))
     (pad 3 thru_hole oval (at 5.08 0 270) (size 1.905 2) (drill 1.1) (layers *.Cu *.Mask)
       (net 1 GND))
@@
       (net 1 GND))
     (pad 2 thru_hole oval (at 2.54 0 270) (size 1.905 2) (drill 1.1) (layers *.Cu *.Mask)
-      (net 31 "Net-(J1-Pad3)"))
+      (net 30 "Net-(J1-Pad3)"))
     (pad 1 thru_hole rect (at 0 0 270) (size 1.905 2) (drill 1.1) (layers *.Cu *.Mask)
-      (net 32 /LED0.1))
+      (net 31 /LED0.1))
     (model ${KISYS3DMOD}/Package_TO_SOT_THT.3dshapes/TO-220-3_Vertical.wrl
       (at (xyz 0 0 0))
@@
     )
     (pad 1 thru_hole rect (at 0 0 270) (size 1.905 2) (drill 1.1) (layers *.Cu *.Mask)
-      (net 29 /LED0.0))
+      (net 28 /LED0.0))
     (pad 2 thru_hole oval (at 2.54 0 270) (size 1.905 2) (drill 1.1) (layers *.Cu *.Mask)
-      (net 30 "Net-(J1-Pad2)"))
+      (net 29 "Net-(J1-Pad2)"))
     (pad 3 thru_hole oval (at 5.08 0 270) (size 1.905 2) (drill 1.1) (layers *.Cu *.Mask)
       (net 1 GND))
@@
       (net 1 GND))
     (pad 6 smd rect (at -2.85 -0.975 180) (size 1.1 0.4) (layers F.Cu F.Paste F.Mask)
-      (net 29 /LED0.0))
+      (net 28 /LED0.0))
     (pad 7 smd rect (at -2.85 -0.325 180) (size 1.1 0.4) (layers F.Cu F.Paste F.Mask)
-      (net 32 /LED0.1))
+      (net 31 /LED0.1))
     (pad 8 smd rect (at -2.85 0.325 180) (size 1.1 0.4) (layers F.Cu F.Paste F.Mask)
-      (net 33 /LED0.2))
+      (net 32 /LED0.2))
     (pad 9 smd rect (at -2.85 0.975 180) (size 1.1 0.4) (layers F.Cu F.Paste F.Mask)
-      (net 41 /LED1.0))
+      (net 40 /LED1.0))
     (pad 10 smd rect (at -2.85 1.625 180) (size 1.1 0.4) (layers F.Cu F.Paste F.Mask)
-      (net 44 /LED1.1))
+      (net 43 /LED1.1))
     (pad 11 smd rect (at -2.85 2.275 180) (size 1.1 0.4) (layers F.Cu F.Paste F.Mask)
-      (net 45 /LED1.2))
+      (net 44 /LED1.2))
     (pad 12 smd rect (at -2.85 2.925 180) (size 1.1 0.4) (layers F.Cu F.Paste F.Mask)
-      (net 36 /LED2.0))
+      (net 35 /LED2.0))
     (pad 13 smd rect (at -2.85 3.575 180) (size 1.1 0.4) (layers F.Cu F.Paste F.Mask)
-      (net 37 /LED2.1))
+      (net 36 /LED2.1))
     (pad 14 smd rect (at -2.85 4.225 180) (size 1.1 0.4) (layers F.Cu F.Paste F.Mask)
       (net 1 GND))
     (pad 15 smd rect (at 2.85 4.225 180) (size 1.1 0.4) (layers F.Cu F.Paste F.Mask)
-      (net 40 /LED2.2))
+      (net 39 /LED2.2))
     (pad 16 smd rect (at 2.85 3.575 180) (size 1.1 0.4) (layers F.Cu F.Paste F.Mask)
       (net 2 "Net-(U2-Pad16)"))
@@
       (net 7 "Net-(U2-Pad21)"))
     (pad 22 smd rect (at 2.85 -0.325 180) (size 1.1 0.4) (layers F.Cu F.Paste F.Mask)
-      (net 28 /TRIGGER))
+      (net 47 Trigger))
     (pad 23 smd rect (at 2.85 -0.975 180) (size 1.1 0.4) (layers F.Cu F.Paste F.Mask)
       (net 1 GND))
@@
       (net 9 /SDA))
     (pad 28 smd rect (at 2.85 -4.225 180) (size 1.1 0.4) (layers F.Cu F.Paste F.Mask)
-      (net 10 +3V3))
+      (net 48 "Net-(U2-Pad28)"))
     (model ${KISYS3DMOD}/Package_SO.3dshapes/TSSOP-28_4.4x9.7mm_P0.65mm.wrl
       (at (xyz 0 0 0))

Commit message: More work on the schematic.
Parts:
- removed J3: Conn_01x04, Connector_PinHeader_1.00mm:PinHeader_1x04_P1.00mm_Vertical
- added C1: 0.1uF, Capacitor_SMD:C_0805_2012Metric_Pad1.29x1.40mm_HandSolder, F.Cu at (54.8, 107.8)
- added C2: 10uF, Capacitor_SMD:C_0805_2012Metric_Pad1.29x1.40mm_HandSolder, F.Cu at (37.6, 98.8)
- added C3: 0.1uF, Capacitor_SMD:C_0805_2012Metric_Pad1.29x1.40mm_HandSolder, F.Cu at (37.6, 93.8)
- added Q10: IRLZ44N, Package_TO_SOT_THT:TO-220-3_Vertical, F.Cu at (236.2, 55.9)
- added Q11: IRLZ44N, Package_TO_SOT_THT:TO-220-3_Vertical, F.Cu at (236.2, 47.0)
- added Q12: IRLZ44N, Package_TO_SOT_THT:TO-220-3_Vertical, F.Cu at (236.2, 38.1)
- added R3: 10k, Resistor_SMD:R_0805_2012Metric_Pad1.29x1.40mm_HandSolder, F.Cu at (63.7, 107.8)
- added R4: 10k, Resistor_SMD:R_0805_2012Metric_Pad1.29x1.40mm_HandSolder, F.Cu at (52.2, 98.9)
- added TP1: Test_Point, Connector_Pin:Pin_D1.0mm_L10.0mm, F.Cu at (163.8, 68.6)
- J1: value Conn_01x04 -> Conn_01x15_Female; footprint Connector_PinHeader_1.00mm:PinHeader_1x04_P1.00mm_Vertical -> Connector_PinHeader_1.00mm:PinHeader_1x15_P1.00mm_Vertical
- J2: value Conn_01x04 -> Conn_01x05_Female; footprint Connector_PinHeader_1.00mm:PinHeader_1x04_P1.00mm_Vertical -> Connector_PinHeader_1.00mm:PinHeader_1x05_P1.00mm_Vertical
- moved J2 185.5 mm to (75.1, 84.9)
- moved U1 87.1 mm to (51.9, 92.1), turned to 90 degrees
- moved R1 77.8 mm to (56.0, 116.7), turned to 270 degrees
- moved R2 77.3 mm to (61.1, 116.7), turned to 270 degrees
- moved U2 44.5 mm to (165.1, 85.1), turned to 90 degrees
- moved Q9 41.9 mm to (236.2, 64.8), turned to 0 degrees
- moved Q8 39.4 mm to (236.2, 73.7), turned to 0 degrees
- moved Q7 36.9 mm to (236.2, 82.5), turned to 0 degrees
- moved Q6 33.0 mm to (236.2, 91.4), turned to 0 degrees
- moved Q5 30.5 mm to (236.2, 100.3), turned to 0 degrees
- moved Q4 28.0 mm to (236.2, 109.2), turned to 0 degrees
- moved J1 25.4 mm to (280.7, 92.7), turned to 0 degrees
- moved Q3 24.2 mm to (236.2, 118.1), turned to 0 degrees
- moved Q2 21.6 mm to (236.2, 127.0), turned to 0 degrees
- moved Q1 19.1 mm to (236.2, 135.9), turned to 0 degrees
Connections:
- J1 pad 1: +12V -> /LED Strips/LED12
- J1 pad 2: Net-(J1-Pad2) -> /LED Strips/LED11
- J1 pad 3: Net-(J1-Pad3) -> /LED Strips/LED10
- J1 pad 4: Net-(J1-Pad4) -> /LED Strips/LED9
- J2 pad 1: +12V -> GND
- J2 pad 2: Net-(J2-Pad2) -> /RESET
- J2 pad 3: Net-(J2-Pad3) -> /BOOT
- J2 pad 4: Net-(J2-Pad4) -> /TX
- Q1 pad 1: /LED0.0 -> /LED_PWM1
- Q1 pad 2: Net-(J1-Pad2) -> /LED Strips/LED1
- Q2 pad 1: /LED0.1 -> /LED_PWM2
- Q2 pad 2: Net-(J1-Pad3) -> /LED Strips/LED2
- Q3 pad 1: /LED0.2 -> /LED_PWM3
- Q3 pad 2: Net-(J1-Pad4) -> /LED Strips/LED3
- Q4 pad 1: /LED1.0 -> /LED_PWM4
- Q4 pad 2: Net-(J2-Pad2) -> /LED Strips/LED4
- Q5 pad 1: /LED1.1 -> /LED_PWM5
- Q5 pad 2: Net-(J2-Pad3) -> /LED Strips/LED5
- Q6 pad 1: /LED1.2 -> /LED_PWM6
- Q6 pad 2: Net-(J2-Pad4) -> /LED Strips/LED6
- Q7 pad 1: /LED2.0 -> /LED_PWM7
- Q7 pad 2: Net-(J3-Pad2) -> /LED Strips/LED7
- Q8 pad 1: /LED2.1 -> /LED_PWM8
- Q8 pad 2: Net-(J3-Pad3) -> /LED Strips/LED8
- Q9 pad 1: /LED2.2 -> /LED_PWM9
- Q9 pad 2: Net-(J3-Pad4) -> /LED Strips/LED9
- U1 pad 1: Net-(U1-Pad1) -> +3V3
- U1 pad 11: Net-(U1-Pad11) -> /RX
- U1 pad 12: Net-(U1-Pad12) -> /TX
- U1 pad 13: Net-(U1-Pad13) -> GND
- U1 pad 15: Net-(U1-Pad15) -> /RESET
- U1 pad 18: Net-(U1-Pad18) -> GND
- U1 pad 8: Net-(U1-Pad8) -> /BOOT
- U1 pad 9: Net-(U1-Pad9) -> GND
- U2 pad 10: /LED1.1 -> /LED_PWM2
- U2 pad 11: /LED1.2 -> /LED_PWM3
- U2 pad 12: /LED2.0 -> /LED_PWM4
- U2 pad 13: /LED2.1 -> /LED_PWM5
- U2 pad 15: /LED2.2 -> /LED_PWM6
- U2 pad 16: Net-(U2-Pad16) -> /LED_PWM7
- U2 pad 17: Net-(U2-Pad17) -> /LED_PWM8
- U2 pad 18: Net-(U2-Pad18) -> /LED_PWM9
- U2 pad 19: Net-(U2-Pad19) -> /LED_PWM10
- U2 pad 20: Net-(U2-Pad20) -> /LED_PWM11
- U2 pad 21: Net-(U2-Pad21) -> /LED_PWM12
- U2 pad 22: Trigger -> /TRIGGER
- U2 pad 28: Net-(U2-Pad28) -> +3V3
- U2 pad 6: /LED0.0 -> Net-(U2-Pad6)
- U2 pad 7: /LED0.1 -> Net-(U2-Pad7)
- U2 pad 8: /LED0.2 -> Net-(U2-Pad8)
- U2 pad 9: /LED1.0 -> /LED_PWM1
