File: hardware/led-strip-controller-esp8266/led-strip-controller-esp8266.sch (KiCad schematic (older format))
At the start: 4 parts, among them U1 ESP-13-WROOM-02, U2 PCA9685PW

Commit message: More work on the schematic.
Parts:
- added C1, C3: 0.1uF, symbol Device:C
- added C2: 10uF, symbol Device:C
- added J4, J5, J6: Conn_01x01_Male, symbol Connector:Conn_01x01_Male
- added JP1: Boot, symbol Jumper:Jumper_2_Open
- added R3, R4: 10k, symbol Device:R
Connections:
- net labels added: +12V, RX, TRIGGER, TX
- net labels removed: Trigger
- wire segments 52 -> 78
- no-connect marks 6 -> 14

Commit message: More work on the schematic.
Parts:
- removed J4, J5, J6: Conn_01x01_Male, symbol Connector:Conn_01x01_Male
- removed JP1: Boot, symbol Jumper:Jumper_2_Open
- added J2: Conn_01x05_Female, Connector_PinHeader_1.00mm:PinHeader_1x05_P1.00mm_Vertical, symbol Connector:Conn_01x05_Female
- added TP1: Test_Point, Connector_Pin:Pin_D1.0mm_L10.0mm, symbol Connector:Test_Point
- C1, C2, C3: footprint (none) -> Capacitor_SMD:C_0805_2012Metric_Pad1.29x1.40mm_HandSolder
- R3, R4: footprint (none) -> Resistor_SMD:R_0805_2012Metric_Pad1.29x1.40mm_HandSolder
Connections:
- net labels added: BOOT, LED_PWM1, LED_PWM10, LED_PWM11, LED_PWM12, LED_PWM2, LED_PWM3, LED_PWM4, LED_PWM5, LED_PWM6, LED_PWM7, LED_PWM8, LED_PWM9, LED_PWM[1..12], RESET
- net labels removed: LED0.0, LED0.1, LED0.2, LED1.0, LED1.1, LED1.2, LED2.0, LED2.1, LED2.2
- wire segments 78 -> 57
- no-connect marks 14 -> 10

Commit message: Add power supply module and power jack.
Parts:
- added J3: Barrel_Jack, Connector_BarrelJack:BarrelJack_Horizontal, symbol Connector:Barrel_Jack
- added U3: R-78HB3.3-0.5, Converter_DCDC:Converter_DCDC_RECOM_R-78HB-0.5_THT, symbol Regulator_Switching:R-78HB3.3-0.5
Connections:
- wire segments 57 -> 61
- no-connect marks 10 -> 11
Other:
- note added: "External connectors"
- note added: "NOTE: needs to be replaced with a\npin-compatible model with high\nenough output current."
- note added: "Power Supply"

Commit message: Add decoupling capacitor to power supply pin of PCA9685.
Parts:
- added C4: 0.1uF, Capacitor_SMD:C_0805_2012Metric_Pad1.29x1.40mm_HandSolder, symbol Device:C
Changed lines of the file:
@@
 U 1 1 5B0DA7D4
 P 6500 2300
-F 0 "U2" H 6500 3478 50  0000 C CNN
-F 1 "PCA9685PW" H 6500 3387 50  0000 C CNN
+F 0 "U2" H 6200 3250 50  0000 C CNN
+F 1 "PCA9685PW" H 6200 3150 50  0000 C CNN
 F 2 "Package_SO:TSSOP-28_4.4x9.7mm_P0.65mm" H 6525 1325 50  0001 L CNN
 F 3 "http://www.nxp.com/documents/data_sheet/PCA9685.pdf" H 6100 3000 50  0001 C CNN
@@
 Power Supply
 NoConn ~ 9450 5700
+$Comp
+L Device:C C4
+U 1 1 5B13F9D0
+P 6650 1300
+F 0 "C4" V 6902 1300 50  0000 C CNN
+F 1 "0.1uF" V 6811 1300 50  0000 C CNN
+F 2 "Capacitor_SMD:C_0805_2012Metric_Pad1.29x1.40mm_HandSolder" H 6688 1150 50  0001 C CNN
+F 3 "~" H 6650 1300 50  0001 C CNN
+	1    6650 1300
+	0    -1   -1   0
+$EndComp
+Connection ~ 6500 1300
+$Comp
+L power:GND #PWR05
+U 1 1 5B13FB86
+P 6800 1300
+F 0 "#PWR05" H 6800 1050 50  0001 C CNN
+F 1 "GND" V 6805 1172 50  0000 R CNN
+F 2 "" H 6800 1300 50  0001 C CNN
+F 3 "" H 6800 1300 50  0001 C CNN
+	1    6800 1300
+	0    -1   -1   0
+$EndComp
 $EndSCHEMATC

Commit message: Add 3.3V rail to external programming interface, and update schematic PDF.
Parts:
- removed J2: Conn_01x05_Female, Connector_PinHeader_1.00mm:PinHeader_1x05_P1.00mm_Vertical, symbol Connector:Conn_01x05_Female
- added J?: Conn_01x06_Female, symbol Connector:Conn_01x06_Female
Connections:
- wire segments 61 -> 62
Changed lines of the file:
@@
 NoConn ~ 7200 1700
 NoConn ~ 7200 1600
-$Comp
-L Connector:Conn_01x05_Female J2
-U 1 1 5B1D05AE
-P 7800 5900
-F 0 "J2" V 7647 6148 50  0000 L CNN
-F 1 "Conn_01x05_Female" V 7738 6148 50  0000 L CNN
-F 2 "Connector_PinHeader_1.00mm:PinHeader_1x05_P1.00mm_Vertical" H 7800 5900 50  0001 C CNN
-F 3 "~" H 7800 5900 50  0001 C CNN
-	1    7800 5900
-	0    1    1    0
-$EndComp
 Text Label 7600 5700 1    50   ~ 0
 RX
@@
 	0    -1   -1   0
 $EndComp
+$Comp
+L Connector:Conn_01x06_Female J?
+U 1 1 5B1424CF
+P 7800 5900
+F 0 "J?" V 7647 6148 50  0000 L CNN
+F 1 "Conn_01x06_Female" V 7900 5600 50  0000 L CNN
+F 2 "" H 7800 5900 50  0001 C CNN
+F 3 "~" H 7800 5900 50  0001 C CNN
+	1    7800 5900
+	0    1    1    0
+$EndComp
+$Comp
+L power:+3.3V #PWR?
+U 1 1 5B1425F3
+P 7500 5450
+F 0 "#PWR?" H 7500 5300 50  0001 C CNN
+F 1 "+3.3V" V 7500 5700 50  0000 C CNN
+F 2 "" H 7500 5450 50  0001 C CNN
+F 3 "" H 7500 5450 50  0001 C CNN
+	1    7500 5450
+	1    0    0    -1
+$EndComp
+Wire Wire Line
+	7500 5700 7500 5450
 $EndSCHEMATC

Commit message: Add TVS diode and new MOSFET array to schematic.
Parts:
- removed J?: Conn_01x06_Female, symbol Connector:Conn_01x06_Female
- added D1: TVS3V3L4U, Package_SO:TSOP-6_1.65x3.05mm_P0.95mm, symbol my-kicad-symbols:TVS3V3L4U
- added J2: Conn_01x05_Female, Connector_PinHeader_1.00mm:PinHeader_1x05_P1.00mm_Vertical, symbol Connector:Conn_01x05_Female
Connections:
- wire segments 62 -> 73
Changed lines of the file:
@@
 NoConn ~ 7200 1700
 NoConn ~ 7200 1600
-Text Label 7600 5700 1    50   ~ 0
+Text Label 6850 5000 0    50   ~ 0
 RX
-Text Label 7700 5700 1    50   ~ 0
+Text Label 6850 5100 0    50   ~ 0
 TX
-Text Label 7800 5700 1    50   ~ 0
+Text Label 6850 5200 0    50   ~ 0
 BOOT
-Text Label 7900 5700 1    50   ~ 0
+Text Label 6850 5300 0    50   ~ 0
 RESET
-Text Label 8000 5700 1    50   ~ 0
+Text Label 6850 5400 0    50   ~ 0
 GND
 $Comp
@@
 	0    1    1    0
 $EndComp
-Wire Wire Line
-	7900 5700 7900 5450
-Wire Wire Line
-	8000 5700 8000 5450
-Wire Wire Line
-	7800 5700 7800 5450
-Wire Wire Line
-	7700 5700 7700 5450
-Wire Wire Line
-	7600 5700 7600 5450
 Text Label 3750 2300 0    50   ~ 0
 RESET
@@
 	0    -1   -1   0
 $EndComp
-Text Notes 8250 5100 0    50   ~ 10
+Text Notes 7700 4600 0    50   ~ 10
 External connectors
 $Comp
@@
 $EndComp
 $Comp
-L Connector:Conn_01x06_Female J?
-U 1 1 5B1424CF
-P 7800 5900
-F 0 "J?" V 7647 6148 50  0000 L CNN
-F 1 "Conn_01x06_Female" V 7900 5600 50  0000 L CNN
-F 2 "" H 7800 5900 50  0001 C CNN
-F 3 "~" H 7800 5900 50  0001 C CNN
-	1    7800 5900
-	0    1    1    0
-$EndComp
-$Comp
-L power:+3.3V #PWR?
-U 1 1 5B1425F3
-P 7500 5450
-F 0 "#PWR?" H 7500 5300 50  0001 C CNN
-F 1 "+3.3V" V 7500 5700 50  0000 C CNN
-F 2 "" H 7500 5450 50  0001 C CNN
-F 3 "" H 7500 5450 50  0001 C CNN
-	1    7500 5450
-	1    0    0    -1
-$EndComp
-Wire Wire Line
-	7500 5700 7500 5450
+L my-kicad-symbols:TVS3V3L4U D1
+U 1 1 5B2E1334
+P 7650 5850
+F 0 "D1" H 7650 6215 50  0000 C CNN
+F 1 "TVS3V3L4U" H 7650 6124 50  0000 C CNN
+F 2 "Package_SO:TSOP-6_1.65x3.05mm_P0.95mm" H 6575 6300 50  0001 C CNN
+F 3 "https://www.infineon.com/dgdl/TVS3V3L4U_rev_2_2.pdf?folderId=db3a30431f848401011fcbf2ab4c04c4&fileId=db3a3043382e837301385be7912532ed" H 6575 6300 50  0001 C CNN
+	1    7650 5850
+	1    0    0    -1
+$EndComp
+$Comp
+L power:GND #PWR0109
+U 1 1 5B2E1489
+P 7650 6200
+F 0 "#PWR0109" H 7650 5950 50  0001 C CNN
+F 1 "GND" H 7655 6027 50  0000 C CNN
+F 2 "" H 7650 6200 50  0001 C CNN
+F 3 "" H 7650 6200 50  0001 C CNN
+	1    7650 6200
+	1    0    0    -1
+$EndComp
+$Comp
+L Connector:Conn_01x05_Female J2
+U 1 1 5B2EA1F5
+P 6650 5200
+F 0 "J2" H 6600 4850 50  0000 C CNN
+F 1 "Conn_01x05_Female" V 6750 5200 50  0000 C CNN
+F 2 "Connector_PinHeader_1.00mm:PinHeader_1x05_P1.00mm_Vertical" H 6650 5200 50  0001 C CNN
+F 3 "~" H 6650 5200 50  0001 C CNN
+	1    6650 5200
+	-1   0    0    1
+$EndComp
+Wire Wire Line
+	6850 5000 7150 5000
+Wire Wire Line
+	6850 5100 7250 5100
+Wire Wire Line
+	6850 5200 8050 5200
+Wire Wire Line
+	7150 5000 7150 5750
+Wire Wire Line
+	7150 5750 7350 5750
+Connection ~ 7150 5000
+Wire Wire Line
+	7150 5000 8300 5000
+Wire Wire Line
+	7250 5100 7250 5950
+Wire Wire Line
+	7250 5950 7350 5950
+Connection ~ 7250 5100
+Wire Wire Line
+	7250 5100 8300 5100
+Wire Wire Line
+	7950 5750 8050 5750
+Wire Wire Line
+	7950 5950 8150 5950
+Wire Wire Line
+	6850 5300 8150 5300
+Wire Wire Line
+	6850 5400 8300 5400
+Wire Wire Line
+	8050 5750 8050 5200
+Connection ~ 8050 5200
+Wire Wire Line
+	8050 5200 8300 5200
+Wire Wire Line
+	8150 5950 8150 5300
+Connection ~ 8150 5300
+Wire Wire Line
+	8150 5300 8300 5300
 $EndSCHEMATC

Commit message: Add status LED and resistor.
Parts:
- added D2: LED, LED_SMD:LED_0805_2012Metric, symbol Device:LED
- added R5: 470, Resistor_SMD:R_0805_2012Metric_Pad1.29x1.40mm_HandSolder, symbol Device:R
Connections:
- wire segments 73 -> 74
- no-connect marks 11 -> 10
Changed lines of the file:
@@
 NoConn ~ 1800 2600
 NoConn ~ 1800 2200
-NoConn ~ 3750 2800
 NoConn ~ 2800 3200
 $Comp
@@
 Wire Wire Line
 	8150 5300 8300 5300
+$Comp
+L Device:R R5
+U 1 1 5B391E96
+P 4250 2800
+F 0 "R5" V 4043 2800 50  0000 C CNN
+F 1 "470" V 4134 2800 50  0000 C CNN
+F 2 "Resistor_SMD:R_0805_2012Metric_Pad1.29x1.40mm_HandSolder" V 4180 2800 50  0001 C CNN
+F 3 "~" H 4250 2800 50  0001 C CNN
+	1    4250 2800
+	0    1    1    0
+$EndComp
+$Comp
+L Device:LED D2
+U 1 1 5B391F79
+P 4550 2800
+F 0 "D2" H 4542 2545 50  0000 C CNN
+F 1 "LED" H 4542 2636 50  0000 C CNN
+F 2 "LED_SMD:LED_0805_2012Metric" H 4550 2800 50  0001 C CNN
+F 3 "~" H 4550 2800 50  0001 C CNN
+	1    4550 2800
+	-1   0    0    1
+$EndComp
+$Comp
+L power:GND #PWR06
+U 1 1 5B39200C
+P 4700 2800
+F 0 "#PWR06" H 4700 2550 50  0001 C CNN
+F 1 "GND" V 4705 2672 50  0000 R CNN
+F 2 "" H 4700 2800 50  0001 C CNN
+F 3 "" H 4700 2800 50  0001 C CNN
+	1    4700 2800
+	0    -1   -1   0
+$EndComp
+Wire Wire Line
+	4100 2800 3750 2800
 $EndSCHEMATC

Commit message: Add a mode/reset button.
Parts:
- added SW1: Mode/Reset, Button_Switch_THT:SW_PUSH_6mm, symbol Switch:SW_Push
Connections:
- wire segments 74 -> 75
- no-connect marks 10 -> 9
Changed lines of the file:
@@
 Text Label 3750 2600 0    50   ~ 0
 TX
-NoConn ~ 3750 2400
 NoConn ~ 3750 2200
 NoConn ~ 3750 2100
@@
 Wire Wire Line
 	4100 2800 3750 2800
+$Comp
+L Switch:SW_Push SW1
+U 1 1 5B3961B5
+P 4500 2400
+F 0 "SW1" H 4500 2685 50  0000 C CNN
+F 1 "Mode/Reset" H 4500 2594 50  0000 C CNN
+F 2 "Button_Switch_THT:SW_PUSH_6mm" H 4500 2600 50  0001 C CNN
+F 3 "" H 4500 2600 50  0001 C CNN
+	1    4500 2400
+	1    0    0    -1
+$EndComp
+$Comp
+L power:GND #PWR0110
+U 1 1 5B396317
+P 4700 2400
+F 0 "#PWR0110" H 4700 2150 50  0001 C CNN
+F 1 "GND" V 4705 2272 50  0000 R CNN
+F 2 "" H 4700 2400 50  0001 C CNN
+F 3 "" H 4700 2400 50  0001 C CNN
+	1    4700 2400
+	0    -1   -1   0
+$EndComp
+Wire Wire Line
+	3750 2400 4300 2400
 $EndSCHEMATC
